Commit message: fix rviz cannot display: modify leg.xacro add joint_state_publisher_node

File: xacro/gazebo.xacro (robot description, xacro)
@@ -116,5 +116,5 @@
     </gazebo>
     <!-- FR leg -->
-    <gazebo reference="rf_hip">
+    <gazebo reference="rf_hip_link">
         <mu1>0.2</mu1>
         <mu2>0.2</mu2>
@@ -140,5 +140,5 @@
     </gazebo>
     <!-- RL leg -->
-    <gazebo reference="lh_hip">
+    <gazebo reference="lh_hip_link">
         <mu1>0.2</mu1>
         <mu2>0.2</mu2>
@@ -164,5 +164,5 @@
     </gazebo>
     <!-- RR leg -->
-    <gazebo reference="rh_hip">
+    <gazebo reference="rh_hip_link">
         <mu1>0.2</mu1>
         <mu2>0.2</mu2>

File: xacro/leg.xacro (robot description, xacro)
@@ -128,5 +128,5 @@
             </inertial>
         </link>
-        <joint name="${name}_foot_joint" type="fixed">0
+        <joint name="${name}_foot_joint" type="fixed">
             <origin rpy="0 0 0" xyz="0 0 ${-(calf_length)}"/>
             <parent link="${name}_lower_leg_link"/>
